File: motortreiber.sch (KiCad schematic (older format))
At the start: 40 parts, among them P15 STP_Y, P16 STP_E0, P17 STP_X, P18 STP_E1, P19 STP_Z, U3 A4988-BO, U4 A4988-BO, U5 A4988-BO, U6 A4988-BO, U7 A4988-BO

Commit message: Added decoupling cap for display supply; Associated most footprints.
Parts:
- renumbered R14 to R18, R15 to R19, R16 to R20, R17 to R21, R18 to R22
Changed lines of the file:
@@
 $EndComp
 $Comp
-L +3,3V #PWR056
+L +3,3V #PWR62
 U 1 1 52E93AEA
 P 3600 1800
-F 0 "#PWR056" H 3600 1760 30  0001 C CNN
+F 0 "#PWR62" H 3600 1760 30  0001 C CNN
 F 1 "+3,3V" H 3600 1910 30  0000 C CNN
 F 2 "" H 3600 1800 60  0000 C CNN
@@
 $EndComp
 $Comp
-L GND #PWR057
+L GND #PWR63
 U 1 1 52E93AF0
 P 3600 1950
-F 0 "#PWR057" H 3600 1950 30  0001 C CNN
+F 0 "#PWR63" H 3600 1950 30  0001 C CNN
 F 1 "GND" H 3600 1880 30  0001 C CNN
 F 2 "" H 3600 1950 60  0000 C CNN
@@
 $EndComp
 $Comp
-L +12V #PWR058
+L +12V #PWR66
 U 1 1 52E93AFC
 P 3650 750
-F 0 "#PWR058" H 3650 700 20  0001 C CNN
+F 0 "#PWR66" H 3650 700 20  0001 C CNN
 F 1 "+12V" H 3650 850 30  0000 C CNN
 F 2 "" H 3650 750 60  0000 C CNN
@@
 $EndComp
 $Comp
-L +3,3V #PWR059
+L +3,3V #PWR58
 U 1 1 52E93B0E
 P 1000 1000
-F 0 "#PWR059" H 1000 960 30  0001 C CNN
+F 0 "#PWR58" H 1000 960 30  0001 C CNN
 F 1 "+3,3V" H 1000 1110 30  0000 C CNN
 F 2 "" H 1000 1000 60  0000 C CNN
@@
 $EndComp
 $Comp
-L +3,3V #PWR060
+L +3,3V #PWR72
 U 1 1 52E93CD6
 P 7000 1800
-F 0 "#PWR060" H 7000 1760 30  0001 C CNN
+F 0 "#PWR72" H 7000 1760 30  0001 C CNN
 F 1 "+3,3V" H 7000 1910 30  0000 C CNN
 F 2 "" H 7000 1800 60  0000 C CNN
@@
 $EndComp
 $Comp
-L GND #PWR061
+L GND #PWR73
 U 1 1 52E93CDC
 P 7000 1950
-F 0 "#PWR061" H 7000 1950 30  0001 C CNN
+F 0 "#PWR73" H 7000 1950 30  0001 C CNN
 F 1 "GND" H 7000 1880 30  0001 C CNN
 F 2 "" H 7000 1950 60  0000 C CNN
@@
 $EndComp
 $Comp
-L +12V #PWR062
+L +12V #PWR76
 U 1 1 52E93CE8
 P 7050 750
-F 0 "#PWR062" H 7050 700 20  0001 C CNN
+F 0 "#PWR76" H 7050 700 20  0001 C CNN
 F 1 "+12V" H 7050 850 30  0000 C CNN
 F 2 "" H 7050 750 60  0000 C CNN
@@
 $EndComp
 $Comp
-L +3,3V #PWR063
+L +3,3V #PWR68
 U 1 1 52E93CFA
 P 4400 1000
-F 0 "#PWR063" H 4400 960 30  0001 C CNN
+F 0 "#PWR68" H 4400 960 30  0001 C CNN
 F 1 "+3,3V" H 4400 1110 30  0000 C CNN
 F 2 "" H 4400 1000 60  0000 C CNN
@@
 $EndComp
 $Comp
-L +3,3V #PWR064
+L +3,3V #PWR80
 U 1 1 52E93D30
 P 10350 1800
-F 0 "#PWR064" H 10350 1760 30  0001 C CNN
+F 0 "#PWR80" H 10350 1760 30  0001 C CNN
 F 1 "+3,3V" H 10350 1910 30  0000 C CNN
 F 2 "" H 10350 1800 60  0000 C CNN
@@
 $EndComp
 $Comp
-L GND #PWR065
+L GND #PWR81
 U 1 1 52E93D36
 P 10350 1950
-F 0 "#PWR065" H 10350 1950 30  0001 C CNN
+F 0 "#PWR81" H 10350 1950 30  0001 C CNN
 F 1 "GND" H 10350 1880 30  0001 C CNN
 F 2 "" H 10350 1950 60  0000 C CNN
@@
 $EndComp
 $Comp
-L +12V #PWR066
+L +12V #PWR82
 U 1 1 52E93D42
 P 10400 750
-F 0 "#PWR066" H 10400 700 20  0001 C CNN
+F 0 "#PWR82" H 10400 700 20  0001 C CNN
 F 1 "+12V" H 10400 850 30  0000 C CNN
 F 2 "" H 10400 750 60  0000 C CNN
@@
 $EndComp
 $Comp
-L +3,3V #PWR067
+L +3,3V #PWR78
 U 1 1 52E93D54
 P 7750 1000
-F 0 "#PWR067" H 7750 960 30  0001 C CNN
+F 0 "#PWR78" H 7750 960 30  0001 C CNN
 F 1 "+3,3V" H 7750 1110 30  0000 C CNN
 F 2 "" H 7750 1000 60  0000 C CNN
@@
 $EndComp
 $Comp
-L +3,3V #PWR068
+L +3,3V #PWR64
 U 1 1 52E93E2A
 P 3600 3550
-F 0 "#PWR068" H 3600 3510 30  0001 C CNN
+F 0 "#PWR64" H 3600 3510 30  0001 C CNN
 F 1 "+3,3V" H 3600 3660 30  0000 C CNN
 F 2 "" H 3600 3550 60  0000 C CNN
@@
 $EndComp
 $Comp
-L GND #PWR069
+L GND #PWR65
 U 1 1 52E93E30
 P 3600 3700
-F 0 "#PWR069" H 3600 3700 30  0001 C CNN
+F 0 "#PWR65" H 3600 3700 30  0001 C CNN
 F 1 "GND" H 3600 3630 30  0001 C CNN
 F 2 "" H 3600 3700 60  0000 C CNN
@@
 $EndComp
 $Comp
-L +12V #PWR070
+L +12V #PWR67
 U 1 1 52E93E3C
 P 3700 2500
-F 0 "#PWR070" H 3700 2450 20  0001 C CNN
+F 0 "#PWR67" H 3700 2450 20  0001 C CNN
 F 1 "+12V" H 3700 2600 30  0000 C CNN
 F 2 "" H 3700 2500 60  0000 C CNN
@@
 $EndComp
 $Comp
-L +3,3V #PWR071
+L +3,3V #PWR59
 U 1 1 52E93E4E
 P 1000 2750
-F 0 "#PWR071" H 1000 2710 30  0001 C CNN
+F 0 "#PWR59" H 1000 2710 30  0001 C CNN
 F 1 "+3,3V" H 1000 2860 30  0000 C CNN
 F 2 "" H 1000 2750 60  0000 C CNN
@@
 $EndComp
 $Comp
-L +3,3V #PWR072
+L +3,3V #PWR74
 U 1 1 52E93E84
 P 7000 3700
-F 0 "#PWR072" H 7000 3660 30  0001 C CNN
+F 0 "#PWR74" H 7000 3660 30  0001 C CNN
 F 1 "+3,3V" H 7000 3810 30  0000 C CNN
 F 2 "" H 7000 3700 60  0000 C CNN
@@
 $EndComp
 $Comp
-L GND #PWR073
+L GND #PWR75
 U 1 1 52E93E8A
 P 7000 3850
-F 0 "#PWR073" H 7000 3850 30  0001 C CNN
+F 0 "#PWR75" H 7000 3850 30  0001 C CNN
 F 1 "GND" H 7000 3780 30  0001 C CNN
 F 2 "" H 7000 3850 60  0000 C CNN
@@
 $EndComp
 $Comp
-L +12V #PWR074
+L +12V #PWR77
 U 1 1 52E93E96
 P 7050 2650
-F 0 "#PWR074" H 7050 2600 20  0001 C CNN
+F 0 "#PWR77" H 7050 2600 20  0001 C CNN
 F 1 "+12V" H 7050 2750 30  0000 C CNN
 F 2 "" H 7050 2650 60  0000 C CNN
@@
 $EndComp
 $Comp
-L +3,3V #PWR075
+L +3,3V #PWR69
 U 1 1 52E93EA8
 P 4400 2900
-F 0 "#PWR075" H 4400 2860 30  0001 C CNN
+F 0 "#PWR69" H 4400 2860 30  0001 C CNN
 F 1 "+3,3V" H 4400 3010 30  0000 C CNN
 F 2 "" H 4400 2900 60  0000 C CNN
@@
 $EndComp
 $Comp
-L R R15
+L R R19
 U 1 1 53525C7D
 P 1600 2050
-F 0 "R15" V 1680 2050 40  0000 C CNN
+F 0 "R19" V 1680 2050 40  0000 C CNN
 F 1 "680" V 1607 2051 40  0000 C CNN
 F 2 "" V 1530 2050 30  0000 C CNN
@@
 $EndComp
 $Comp
-L GND #PWR076
+L GND #PWR61
 U 1 1 53525C8F
 P 1600 2350
-F 0 "#PWR076" H 1600 2350 30  0001 C CNN
+F 0 "#PWR61" H 1600 2350 30  0001 C CNN
 F 1 "GND" H 1600 2280 30  0001 C CNN
 F 2 "" H 1600 2350 60  0000 C CNN
@@
 	1600 2350 1600 2300
 $Comp
-L R R14
+L R R18
 U 1 1 53525D19
 P 1550 3800
-F 0 "R14" V 1630 3800 40  0000 C CNN
+F 0 "R18" V 1630 3800 40  0000 C CNN
 F 1 "680" V 1557 3801 40  0000 C CNN
 F 2 "" V 1480 3800 30  0000 C CNN
@@
 $EndComp
 $Comp
-L GND #PWR077
+L GND #PWR60
 U 1 1 53525D1F
 P 1550 4100
-F 0 "#PWR077" H 1550 4100 30  0001 C CNN
+F 0 "#PWR60" H 1550 4100 30  0001 C CNN
 F 1 "GND" H 1550 4030 30  0001 C CNN
 F 2 "" H 1550 4100 60  0000 C CNN
@@
 	1550 4100 1550 4050
 $Comp
-L R R16
+L R R20
 U 1 1 53525D26
 P 4950 3950
-F 0 "R16" V 5030 3950 40  0000 C CNN
+F 0 "R20" V 5030 3950 40  0000 C CNN
 F 1 "680" V 4957 3951 40  0000 C CNN
 F 2 "" V 4880 3950 30  0000 C CNN
@@
 $EndComp
 $Comp
-L GND #PWR078
+L GND #PWR70
 U 1 1 53525D2C
 P 4950 4250
-F 0 "#PWR078" H 4950 4250 30  0001 C CNN
+F 0 "#PWR70" H 4950 4250 30  0001 C CNN
 F 1 "GND" H 4950 4180 30  0001 C CNN
 F 2 "" H 4950 4250 60  0000 C CNN
@@
 	4950 4250 4950 4200
 $Comp
-L R R17
+L R R21
 U 1 1 53525D33
 P 5000 2050
-F 0 "R17" V 5080 2050 40  0000 C CNN
+F 0 "R21" V 5080 2050 40  0000 C CNN
 F 1 "680" V 5007 2051 40  0000 C CNN
 F 2 "" V 4930 2050 30  0000 C CNN
@@
 $EndComp
 $Comp
-L GND #PWR079
+L GND #PWR71
 U 1 1 53525D39
 P 5000 2350
-F 0 "#PWR079" H 5000 2350 30  0001 C CNN
+F 0 "#PWR71" H 5000 2350 30  0001 C CNN
 F 1 "GND" H 5000 2280 30  0001 C CNN
 F 2 "" H 5000 2350 60  0000 C CNN
@@
 	5000 2350 5000 2300
 $Comp
-L R R18
+L R R22
 U 1 1 53525D40
 P 8350 2050
-F 0 "R18" V 8430 2050 40  0000 C CNN
+F 0 "R22" V 8430 2050 40  0000 C CNN
 F 1 "680" V 8357 2051 40  0000 C CNN
 F 2 "" V 8280 2050 30  0000 C CNN
@@
 $EndComp
 $Comp
-L GND #PWR080
+L GND #PWR79
 U 1 1 53525D46
 P 8350 2350
-F 0 "#PWR080" H 8350 2350 30  0001 C CNN
+F 0 "#PWR79" H 8350 2350 30  0001 C CNN
 F 1 "GND" H 8350 2280 30  0001 C CNN
 F 2 "" H 8350 2350 60  0000 C CNN

Commit message: Added status LEDs for 5V and 12V power
Parts:
- renumbered C17 to C18, C18 to C19, C19 to C20, C20 to C21, C21 to C22, D3 to D5, D4 to D6, D5 to D7, D6 to D8, D7 to D9, R18 to R20, R19 to R21, R20 to R22, R21 to R23, R22 to R24
Changed lines of the file:
@@
 $EndComp
 $Comp
-L +3,3V #PWR058
+L +3,3V #PWR66
 U 1 1 52E93AEA
 P 3600 1800
-F 0 "#PWR058" H 3600 1760 30  0001 C CNN
+F 0 "#PWR66" H 3600 1760 30  0001 C CNN
 F 1 "+3,3V" H 3600 1910 30  0000 C CNN
 F 2 "" H 3600 1800 60  0000 C CNN
@@
 $EndComp
 $Comp
-L GND #PWR059
+L GND #PWR67
 U 1 1 52E93AF0
 P 3600 1950
-F 0 "#PWR059" H 3600 1950 30  0001 C CNN
+F 0 "#PWR67" H 3600 1950 30  0001 C CNN
 F 1 "GND" H 3600 1880 30  0001 C CNN
 F 2 "" H 3600 1950 60  0000 C CNN
@@
 $EndComp
 $Comp
-L CP1 C17
+L CP1 C18
 U 1 1 52E93AF6
 P 3650 950
-F 0 "C17" H 3700 1050 50  0000 L CNN
+F 0 "C18" H 3700 1050 50  0000 L CNN
 F 1 "100uF" H 3700 850 50  0000 L CNN
 F 2 "~" H 3650 950 60  0000 C CNN
@@
 $EndComp
 $Comp
-L +12V #PWR060
+L +12V #PWR70
 U 1 1 52E93AFC
 P 3650 750
-F 0 "#PWR060" H 3650 700 20  0001 C CNN
+F 0 "#PWR70" H 3650 700 20  0001 C CNN
 F 1 "+12V" H 3650 850 30  0000 C CNN
 F 2 "" H 3650 750 60  0000 C CNN
@@
 $EndComp
 $Comp
-L +3,3V #PWR061
+L +3,3V #PWR62
 U 1 1 52E93B0E
 P 1000 1000
-F 0 "#PWR061" H 1000 960 30  0001 C CNN
+F 0 "#PWR62" H 1000 960 30  0001 C CNN
 F 1 "+3,3V" H 1000 1110 30  0000 C CNN
 F 2 "" H 1000 1000 60  0000 C CNN
@@
 $EndComp
 $Comp
-L +3,3V #PWR062
+L +3,3V #PWR76
 U 1 1 52E93CD6
 P 7000 1800
-F 0 "#PWR062" H 7000 1760 30  0001 C CNN
+F 0 "#PWR76" H 7000 1760 30  0001 C CNN
 F 1 "+3,3V" H 7000 1910 30  0000 C CNN
 F 2 "" H 7000 1800 60  0000 C CNN
@@
 $EndComp
 $Comp
-L GND #PWR063
+L GND #PWR77
 U 1 1 52E93CDC
 P 7000 1950
-F 0 "#PWR063" H 7000 1950 30  0001 C CNN
+F 0 "#PWR77" H 7000 1950 30  0001 C CNN
 F 1 "GND" H 7000 1880 30  0001 C CNN
 F 2 "" H 7000 1950 60  0000 C CNN
@@
 $EndComp
 $Comp
-L CP1 C19
+L CP1 C20
 U 1 1 52E93CE2
 P 7050 950
-F 0 "C19" H 7100 1050 50  0000 L CNN
+F 0 "C20" H 7100 1050 50  0000 L CNN
 F 1 "100uF" H 7100 850 50  0000 L CNN
 F 2 "~" H 7050 950 60  0000 C CNN
@@
 $EndComp
 $Comp
-L +12V #PWR064
+L +12V #PWR80
 U 1 1 52E93CE8
 P 7050 750
-F 0 "#PWR064" H 7050 700 20  0001 C CNN
+F 0 "#PWR80" H 7050 700 20  0001 C CNN
 F 1 "+12V" H 7050 850 30  0000 C CNN
 F 2 "" H 7050 750 60  0000 C CNN
@@
 $EndComp
 $Comp
-L +3,3V #PWR065
+L +3,3V #PWR72
 U 1 1 52E93CFA
 P 4400 1000
-F 0 "#PWR065" H 4400 960 30  0001 C CNN
+F 0 "#PWR72" H 4400 960 30  0001 C CNN
 F 1 "+3,3V" H 4400 1110 30  0000 C CNN
 F 2 "" H 4400 1000 60  0000 C CNN
@@
 $EndComp
 $Comp
-L +3,3V #PWR066
+L +3,3V #PWR84
 U 1 1 52E93D30
 P 10350 1800
-F 0 "#PWR066" H 10350 1760 30  0001 C CNN
+F 0 "#PWR84" H 10350 1760 30  0001 C CNN
 F 1 "+3,3V" H 10350 1910 30  0000 C CNN
 F 2 "" H 10350 1800 60  0000 C CNN
@@
 $EndComp
 $Comp
-L GND #PWR067
+L GND #PWR85
 U 1 1 52E93D36
 P 10350 1950
-F 0 "#PWR067" H 10350 1950 30  0001 C CNN
+F 0 "#PWR85" H 10350 1950 30  0001 C CNN
 F 1 "GND" H 10350 1880 30  0001 C CNN
 F 2 "" H 10350 1950 60  0000 C CNN
@@
 $EndComp
 $Comp
-L CP1 C21
+L CP1 C22
 U 1 1 52E93D3C
 P 10400 950
-F 0 "C21" H 10450 1050 50  0000 L CNN
+F 0 "C22" H 10450 1050 50  0000 L CNN
 F 1 "100uF" H 10450 850 50  0000 L CNN
 F 2 "~" H 10400 950 60  0000 C CNN
@@
 $EndComp
 $Comp
-L +12V #PWR068
+L +12V #PWR86
 U 1 1 52E93D42
 P 10400 750
-F 0 "#PWR068" H 10400 700 20  0001 C CNN
+F 0 "#PWR86" H 10400 700 20  0001 C CNN
 F 1 "+12V" H 10400 850 30  0000 C CNN
 F 2 "" H 10400 750 60  0000 C CNN
@@
 $EndComp
 $Comp
-L +3,3V #PWR069
+L +3,3V #PWR82
 U 1 1 52E93D54
 P 7750 1000
-F 0 "#PWR069" H 7750 960 30  0001 C CNN
+F 0 "#PWR82" H 7750 960 30  0001 C CNN
 F 1 "+3,3V" H 7750 1110 30  0000 C CNN
 F 2 "" H 7750 1000 60  0000 C CNN
@@
 $EndComp
 $Comp
-L +3,3V #PWR070
+L +3,3V #PWR68
 U 1 1 52E93E2A
 P 3600 3550
-F 0 "#PWR070" H 3600 3510 30  0001 C CNN
+F 0 "#PWR68" H 3600 3510 30  0001 C CNN
 F 1 "+3,3V" H 3600 3660 30  0000 C CNN
 F 2 "" H 3600 3550 60  0000 C CNN
@@
 $EndComp
 $Comp
-L GND #PWR071
+L GND #PWR69
 U 1 1 52E93E30
 P 3600 3700
-F 0 "#PWR071" H 3600 3700 30  0001 C CNN
+F 0 "#PWR69" H 3600 3700 30  0001 C CNN
 F 1 "GND" H 3600 3630 30  0001 C CNN
 F 2 "" H 3600 3700 60  0000 C CNN
@@
 $EndComp
 $Comp
-L CP1 C18
+L CP1 C19
 U 1 1 52E93E36
 P 3700 2700
-F 0 "C18" H 3750 2800 50  0000 L CNN
+F 0 "C19" H 3750 2800 50  0000 L CNN
 F 1 "100uF" H 3750 2600 50  0000 L CNN
 F 2 "~" H 3700 2700 60  0000 C CNN
@@
 $EndComp
 $Comp
-L +12V #PWR072
+L +12V #PWR71
 U 1 1 52E93E3C
 P 3700 2500
-F 0 "#PWR072" H 3700 2450 20  0001 C CNN
+F 0 "#PWR71" H 3700 2450 20  0001 C CNN
 F 1 "+12V" H 3700 2600 30  0000 C CNN
 F 2 "" H 3700 2500 60  0000 C CNN
@@
 $EndComp
 $Comp
-L +3,3V #PWR073
+L +3,3V #PWR63
 U 1 1 52E93E4E
 P 1000 2750
-F 0 "#PWR073" H 1000 2710 30  0001 C CNN
+F 0 "#PWR63" H 1000 2710 30  0001 C CNN
 F 1 "+3,3V" H 1000 2860 30  0000 C CNN
 F 2 "" H 1000 2750 60  0000 C CNN
@@
 $EndComp
 $Comp
-L +3,3V #PWR074
+L +3,3V #PWR78
 U 1 1 52E93E84
 P 7000 3700
-F 0 "#PWR074" H 7000 3660 30  0001 C CNN
+F 0 "#PWR78" H 7000 3660 30  0001 C CNN
 F 1 "+3,3V" H 7000 3810 30  0000 C CNN
 F 2 "" H 7000 3700 60  0000 C CNN
@@
 $EndComp
 $Comp
-L GND #PWR075
+L GND #PWR79
 U 1 1 52E93E8A
 P 7000 3850
-F 0 "#PWR075" H 7000 3850 30  0001 C CNN
+F 0 "#PWR79" H 7000 3850 30  0001 C CNN
 F 1 "GND" H 7000 3780 30  0001 C CNN
 F 2 "" H 7000 3850 60  0000 C CNN
@@
 $EndComp
 $Comp
-L CP1 C20
+L CP1 C21
 U 1 1 52E93E90
 P 7050 2850
-F 0 "C20" H 7100 2950 50  0000 L CNN
+F 0 "C21" H 7100 2950 50  0000 L CNN
 F 1 "100uF" H 7100 2750 50  0000 L CNN
 F 2 "~" H 7050 2850 60  0000 C CNN
@@
 $EndComp
 $Comp
-L +12V #PWR076
+L +12V #PWR81
 U 1 1 52E93E96
 P 7050 2650
-F 0 "#PWR076" H 7050 2600 20  0001 C CNN
+F 0 "#PWR81" H 7050 2600 20  0001 C CNN
 F 1 "+12V" H 7050 2750 30  0000 C CNN
 F 2 "" H 7050 2650 60  0000 C CNN
@@
 $EndComp
 $Comp
-L +3,3V #PWR077
+L +3,3V #PWR73
 U 1 1 52E93EA8
 P 4400 2900
-F 0 "#PWR077" H 4400 2860 30  0001 C CNN
+F 0 "#PWR73" H 4400 2860 30  0001 C CNN
 F 1 "+3,3V" H 4400 3010 30  0000 C CNN
 F 2 "" H 4400 2900 60  0000 C CNN
@@
 	8800 1700 8850 1700
 $Comp
-L LED D4
+L LED D6
 U 1 1 53525C3D
 P 1600 1600
-F 0 "D4" H 1600 1700 50  0000 C CNN
+F 0 "D6" H 1600 1700 50  0000 C CNN
 F 1 "ST-Y" H 1600 1500 50  0000 C CNN
 F 2 "" H 1600 1600 60  0000 C CNN
@@
 $EndComp
 $Comp
-L LED D6
+L LED D8
 U 1 1 53525C4F
 P 5000 1600
-F 0 "D6" H 5000 1700 50  0000 C CNN
+F 0 "D8" H 5000 1700 50  0000 C CNN
 F 1 "ST-X" H 5000 1500 50  0000 C CNN
 F 2 "" H 5000 1600 60  0000 C CNN
@@
 $EndComp
 $Comp
-L LED D7
+L LED D9
 U 1 1 53525C5A
 P 8350 1600
-F 0 "D7" H 8350 1700 50  0000 C CNN
+F 0 "D9" H 8350 1700 50  0000 C CNN
 F 1 "ST-Z" H 8350 1500 50  0000 C CNN
 F 2 "" H 8350 1600 60  0000 C CNN
@@
 $EndComp
 $Comp
-L LED D5
+L LED D7
 U 1 1 53525C65
 P 4950 3500
-F 0 "D5" H 4950 3600 50  0000 C CNN
+F 0 "D7" H 4950 3600 50  0000 C CNN
 F 1 "ST-E1" H 4950 3400 50  0000 C CNN
 F 2 "" H 4950 3500 60  0000 C CNN
@@
 $EndComp
 $Comp
-L LED D3
+L LED D5
 U 1 1 53525C70
 P 1550 3350
-F 0 "D3" H 1550 3450 50  0000 C CNN
+F 0 "D5" H 1550 3450 50  0000 C CNN
 F 1 "ST-E0" H 1550 3250 50  0000 C CNN
 F 2 "" H 1550 3350 60  0000 C CNN
@@
 $EndComp
 $Comp
-L R R19
+L R R21
 U 1 1 53525C7D
 P 1600 2050
-F 0 "R19" V 1680 2050 40  0000 C CNN
+F 0 "R21" V 1680 2050 40  0000 C CNN
 F 1 "680" V 1607 2051 40  0000 C CNN
 F 2 "" V 1530 2050 30  0000 C CNN
@@
 $EndComp
 $Comp
-L GND #PWR078
+L GND #PWR65
 U 1 1 53525C8F
 P 1600 2350
-F 0 "#PWR078" H 1600 2350 30  0001 C CNN
+F 0 "#PWR65" H 1600 2350 30  0001 C CNN
 F 1 "GND" H 1600 2280 30  0001 C CNN
 F 2 "" H 1600 2350 60  0000 C CNN
@@
 	1600 2350 1600 2300
 $Comp
-L R R18
+L R R20
 U 1 1 53525D19
 P 1550 3800
-F 0 "R18" V 1630 3800 40  0000 C CNN
+F 0 "R20" V 1630 3800 40  0000 C CNN
 F 1 "680" V 1557 3801 40  0000 C CNN
 F 2 "" V 1480 3800 30  0000 C CNN
@@
 $EndComp
 $Comp
-L GND #PWR079
+L GND #PWR64
 U 1 1 53525D1F
 P 1550 4100
-F 0 "#PWR079" H 1550 4100 30  0001 C CNN
+F 0 "#PWR64" H 1550 4100 30  0001 C CNN
 F 1 "GND" H 1550 4030 30  0001 C CNN
 F 2 "" H 1550 4100 60  0000 C CNN
@@
 	1550 4100 1550 4050
 $Comp
-L R R20
+L R R22
 U 1 1 53525D26
 P 4950 3950
-F 0 "R20" V 5030 3950 40  0000 C CNN
+F 0 "R22" V 5030 3950 40  0000 C CNN
 F 1 "680" V 4957 3951 40  0000 C CNN
 F 2 "" V 4880 3950 30  0000 C CNN
@@
 $EndComp
 $Comp
-L GND #PWR080
+L GND #PWR74
 U 1 1 53525D2C
 P 4950 4250
-F 0 "#PWR080" H 4950 4250 30  0001 C CNN
+F 0 "#PWR74" H 4950 4250 30  0001 C CNN
 F 1 "GND" H 4950 4180 30  0001 C CNN
 F 2 "" H 4950 4250 60  0000 C CNN
@@
 	4950 4250 4950 4200
 $Comp
-L R R21
+L R R23
 U 1 1 53525D33
 P 5000 2050
-F 0 "R21" V 5080 2050 40  0000 C CNN
+F 0 "R23" V 5080 2050 40  0000 C CNN
 F 1 "680" V 5007 2051 40  0000 C CNN
 F 2 "" V 4930 2050 30  0000 C CNN
@@
 $EndComp
 $Comp
-L GND #PWR081
+L GND #PWR75
 U 1 1 53525D39
 P 5000 2350
-F 0 "#PWR081" H 5000 2350 30  0001 C CNN
+F 0 "#PWR75" H 5000 2350 30  0001 C CNN
 F 1 "GND" H 5000 2280 30  0001 C CNN
 F 2 "" H 5000 2350 60  0000 C CNN
@@
 	5000 2350 5000 2300
 $Comp
-L R R22
+L R R24
 U 1 1 53525D40
 P 8350 2050
-F 0 "R22" V 8430 2050 40  0000 C CNN
+F 0 "R24" V 8430 2050 40  0000 C CNN
 F 1 "680" V 8357 2051 40  0000 C CNN
 F 2 "" V 8280 2050 30  0000 C CNN
@@
 $EndComp
 $Comp
-L GND #PWR082
+L GND #PWR83
 U 1 1 53525D46
 P 8350 2350
-F 0 "#PWR082" H 8350 2350 30  0001 C CNN
+F 0 "#PWR83" H 8350 2350 30  0001 C CNN
 F 1 "GND" H 8350 2280 30  0001 C CNN
 F 2 "" H 8350 2350 60  0000 C CNN
