File: heater-fan-driver.sch (KiCad schematic (older format))
At the start: 35 parts, among them P20 EXTR, P21 HIC_0, P22 HEATBED, P23 HIC_1, P24 FAN_0, P25 FAN_1, P26 LOC_0, P27 LOC_1, Q1 IRL1404, Q2 IRL1404, Q3 IRL1404, Q4 IRL1404, U10 ULN_2003_A, U8 MCP14E10, U9 MCP14E10

Commit message: Added status LEDs for 5V and 12V power
Parts:
- renumbered D8 to D10, D9 to D11, D10 to D12, D11 to D13, D12 to D14, D13 to D15, D14 to D16, D15 to D17, D16 to D18, D17 to D19, D18 to D20, D19 to D21, R23 to R25, R24 to R26, R25 to R27, R26 to R28, R27 to R29, R28 to R30, R29 to R31, R30 to R32
Changed lines of the file:
@@
 NoConn ~ 1500 3100
 $Comp
-L +12V #PWR083
+L +12V #PWR87
 U 1 1 534EA91F
 P 2250 2550
-F 0 "#PWR083" H 2250 2500 20  0001 C CNN
+F 0 "#PWR87" H 2250 2500 20  0001 C CNN
 F 1 "+12V" H 2250 2650 30  0000 C CNN
 F 2 "" H 2250 2550 60  0000 C CNN
@@
 $EndComp
 $Comp
-L GND #PWR084
+L GND #PWR88
 U 1 1 534EA925
 P 2250 3450
-F 0 "#PWR084" H 2250 3450 30  0001 C CNN
+F 0 "#PWR88" H 2250 3450 30  0001 C CNN
 F 1 "GND" H 2250 3380 30  0001 C CNN
 F 2 "" H 2250 3450 60  0000 C CNN
@@
 NoConn ~ 1500 5400
 $Comp
-L +12V #PWR085
+L +12V #PWR89
 U 1 1 534EA949
 P 2250 4850
-F 0 "#PWR085" H 2250 4800 20  0001 C CNN
+F 0 "#PWR89" H 2250 4800 20  0001 C CNN
 F 1 "+12V" H 2250 4950 30  0000 C CNN
 F 2 "" H 2250 4850 60  0000 C CNN
@@
 $EndComp
 $Comp
-L GND #PWR086
+L GND #PWR90
 U 1 1 534EA94F
 P 2250 5750
-F 0 "#PWR086" H 2250 5750 30  0001 C CNN
+F 0 "#PWR90" H 2250 5750 30  0001 C CNN
 F 1 "GND" H 2250 5680 30  0001 C CNN
 F 2 "" H 2250 5750 60  0000 C CNN
@@
 $EndComp
 $Comp
-L GND #PWR087
+L GND #PWR92
 U 1 1 534EC0D7
 P 3850 3200
-F 0 "#PWR087" H 3850 3200 30  0001 C CNN
+F 0 "#PWR92" H 3850 3200 30  0001 C CNN
 F 1 "GND" H 3850 3130 30  0001 C CNN
 F 2 "" H 3850 3200 60  0000 C CNN
@@
 	3850 2500 3850 2650
 $Comp
-L +12V #PWR088
+L +12V #PWR91
 U 1 1 534EC0F8
 P 3850 2100
-F 0 "#PWR088" H 3850 2050 20  0001 C CNN
+F 0 "#PWR91" H 3850 2050 20  0001 C CNN
 F 1 "+12V" H 3850 2200 30  0000 C CNN
 F 2 "" H 3850 2100 60  0000 C CNN
@@
 $EndComp
 $Comp
-L GND #PWR089
+L GND #PWR98
 U 1 1 534EC131
 P 4850 3850
-F 0 "#PWR089" H 4850 3850 30  0001 C CNN
+F 0 "#PWR98" H 4850 3850 30  0001 C CNN
 F 1 "GND" H 4850 3780 30  0001 C CNN
 F 2 "" H 4850 3850 60  0000 C CNN
@@
 	4850 3150 4850 3300
 $Comp
-L +12V #PWR090
+L +12V #PWR97
 U 1 1 534EC139
 P 4850 2750
-F 0 "#PWR090" H 4850 2700 20  0001 C CNN
+F 0 "#PWR97" H 4850 2700 20  0001 C CNN
 F 1 "+12V" H 4850 2850 30  0000 C CNN
 F 2 "" H 4850 2750 60  0000 C CNN
@@
 $EndComp
 $Comp
-L GND #PWR091
+L GND #PWR94
 U 1 1 534EC15C
 P 3850 5500
-F 0 "#PWR091" H 3850 5500 30  0001 C CNN
+F 0 "#PWR94" H 3850 5500 30  0001 C CNN
 F 1 "GND" H 3850 5430 30  0001 C CNN
 F 2 "" H 3850 5500 60  0000 C CNN
@@
 	3850 4800 3850 4950
 $Comp
-L +12V #PWR092
+L +12V #PWR93
 U 1 1 534EC164
 P 3850 4400
-F 0 "#PWR092" H 3850 4350 20  0001 C CNN
+F 0 "#PWR93" H 3850 4350 20  0001 C CNN
 F 1 "+12V" H 3850 4500 30  0000 C CNN
 F 2 "" H 3850 4400 60  0000 C CNN
@@
 $EndComp
 $Comp
-L GND #PWR093
+L GND #PWR96
 U 1 1 534EC178
 P 4650 6100
-F 0 "#PWR093" H 4650 6100 30  0001 C CNN
+F 0 "#PWR96" H 4650 6100 30  0001 C CNN
 F 1 "GND" H 4650 6030 30  0001 C CNN
 F 2 "" H 4650 6100 60  0000 C CNN
@@
 	4650 6100 4650 5950
 $Comp
-L +12V #PWR094
+L +12V #PWR95
 U 1 1 534EC180
 P 4650 5050
-F 0 "#PWR094" H 4650 5000 20  0001 C CNN
+F 0 "#PWR95" H 4650 5000 20  0001 C CNN
 F 1 "+12V" H 4650 5150 30  0000 C CNN
 F 2 "" H 4650 5050 60  0000 C CNN
@@
 $EndComp
 $Comp
-L GND #PWR095
+L GND #PWR100
 U 1 1 534EF1D5
 P 6800 5000
-F 0 "#PWR095" H 6800 5000 30  0001 C CNN
+F 0 "#PWR100" H 6800 5000 30  0001 C CNN
 F 1 "GND" H 6800 4930 30  0001 C CNN
 F 2 "" H 6800 5000 60  0000 C CNN
@@
 	6800 4950 6850 4950
 $Comp
-L +12V #PWR096
+L +12V #PWR101
 U 1 1 534EF1FB
 P 7950 5000
-F 0 "#PWR096" H 7950 4950 20  0001 C CNN
+F 0 "#PWR101" H 7950 4950 20  0001 C CNN
 F 1 "+12V" H 7950 5100 30  0000 C CNN
 F 2 "" H 7950 5000 60  0000 C CNN
@@
 	6800 4800 6850 4800
 $Comp
-L GND #PWR097
+L GND #PWR99
 U 1 1 534EF2C3
 P 6250 5000
-F 0 "#PWR097" H 6250 5000 30  0001 C CNN
+F 0 "#PWR99" H 6250 5000 30  0001 C CNN
 F 1 "GND" H 6250 4930 30  0001 C CNN
 F 2 "" H 6250 5000 60  0000 C CNN
@@
 $EndComp
 $Comp
-L +12V #PWR098
+L +12V #PWR102
 U 1 1 534EF366
 P 8800 2850
-F 0 "#PWR098" H 8800 2800 20  0001 C CNN
+F 0 "#PWR102" H 8800 2800 20  0001 C CNN
 F 1 "+12V" H 8800 2950 30  0000 C CNN
 F 2 "" H 8800 2850 60  0000 C CNN
@@
 IN_HIC_1
 $Comp
-L LED D8
+L LED D10
 U 1 1 53500700
 P 3150 2400
-F 0 "D8" H 3150 2500 50  0000 C CNN
+F 0 "D10" H 3150 2500 50  0000 C CNN
 F 1 "EXTR" H 3150 2300 50  0000 C CNN
 F 2 "0805" H 3150 2400 60  0000 C CNN
@@
 $EndComp
 $Comp
-L R R23
+L R R25
 U 1 1 53500760
 P 3450 2150
-F 0 "R23" V 3530 2150 40  0000 C CNN
+F 0 "R25" V 3530 2150 40  0000 C CNN
 F 1 "4.7k" V 3457 2151 40  0000 C CNN
 F 2 "" V 3380 2150 30  0000 C CNN
@@
 Connection ~ 3850 2600
 $Comp
-L LED D13
+L LED D15
 U 1 1 535007F1
 P 4150 3050
-F 0 "D13" H 4150 3150 50  0000 C CNN
+F 0 "D15" H 4150 3150 50  0000 C CNN
 F 1 "HB" H 4150 2950 50  0000 C CNN
 F 2 "" H 4150 3050 60  0000 C CNN
@@
 $EndComp
 $Comp
-L R R26
+L R R28
 U 1 1 535007F7
 P 4450 2800
-F 0 "R26" V 4530 2800 40  0000 C CNN
+F 0 "R28" V 4530 2800 40  0000 C CNN
 F 1 "4.7k" V 4457 2801 40  0000 C CNN
 F 2 "" V 4380 2800 30  0000 C CNN
@@
 	3300 3500 4550 3500
 $Comp
-L LED D9
+L LED D11
 U 1 1 535008DF
 P 3150 4700
-F 0 "D9" H 3150 4800 50  0000 C CNN
+F 0 "D11" H 3150 4800 50  0000 C CNN
 F 1 "HIC0" H 3150 4600 50  0000 C CNN
 F 2 "" H 3150 4700 60  0000 C CNN
@@
 $EndComp
 $Comp
-L R R24
+L R R26
 U 1 1 535008E5
 P 3450 4450
-F 0 "R24" V 3530 4450 40  0000 C CNN
+F 0 "R26" V 3530 4450 40  0000 C CNN
 F 1 "4.7k" V 3457 4451 40  0000 C CNN
 F 2 "" V 3380 4450 30  0000 C CNN
@@
 Connection ~ 3850 4450
 $Comp
-L LED D12
+L LED D14
 U 1 1 535008F7
 P 4100 5350
-F 0 "D12" H 4100 5450 50  0000 C CNN
+F 0 "D14" H 4100 5450 50  0000 C CNN
 F 1 "HIC1" H 4100 5250 50  0000 C CNN
 F 2 "" H 4100 5350 60  0000 C CNN
@@
 $EndComp
 $Comp
-L R R25
+L R R27
 U 1 1 535008FD
 P 4400 5100
-F 0 "R25" V 4480 5100 40  0000 C CNN
+F 0 "R27" V 4480 5100 40  0000 C CNN
 F 1 "4.7k" V 4407 5101 40  0000 C CNN
 F 2 "" V 4330 5100 30  0000 C CNN
@@
 Connection ~ 3850 2150
 $Comp
-L LED D19
+L LED D21
 U 1 1 53500962
 P 8650 3750
-F 0 "D19" H 8650 3850 50  0000 C CNN
+F 0 "D21" H 8650 3850 50  0000 C CNN
 F 1 "LOC1" H 8650 3650 50  0000 C CNN
 F 2 "" H 8650 3750 60  0000 C CNN
@@
 $EndComp
 $Comp
-L LED D18
+L LED D20
 U 1 1 5350096D
 P 8450 3750
-F 0 "D18" H 8450 3850 50  0000 C CNN
+F 0 "D20" H 8450 3850 50  0000 C CNN
 F 1 "LOC0" H 8450 3650 50  0000 C CNN
 F 2 "" H 8450 3750 60  0000 C CNN
@@
 $EndComp
 $Comp
-L LED D17
+L LED D19
 U 1 1 53500978
 P 8250 3750
-F 0 "D17" H 8250 3850 50  0000 C CNN
+F 0 "D19" H 8250 3850 50  0000 C CNN
 F 1 "FAN1" H 8250 3650 50  0000 C CNN
 F 2 "" H 8250 3750 60  0000 C CNN
@@
 $EndComp
 $Comp
-L LED D16
+L LED D18
 U 1 1 53500983
 P 8050 3750
-F 0 "D16" H 8050 3850 50  0000 C CNN
+F 0 "D18" H 8050 3850 50  0000 C CNN
 F 1 "FAN0" H 8050 3650 50  0000 C CNN
 F 2 "" H 8050 3750 60  0000 C CNN
@@
 Connection ~ 8250 2950
 $Comp
-L R R27
+L R R29
 U 1 1 53500AE3
 P 8050 3250
-F 0 "R27" V 8130 3250 40  0000 C CNN
+F 0 "R29" V 8130 3250 40  0000 C CNN
 F 1 "4.7k" V 8057 3251 40  0000 C CNN
 F 2 "" V 7980 3250 30  0000 C CNN
@@
 	8800 2850 8800 5050
 $Comp
-L R R28
+L R R30
 U 1 1 53500D59
 P 8250 3250
-F 0 "R28" V 8330 3250 40  0000 C CNN
+F 0 "R30" V 8330 3250 40  0000 C CNN
 F 1 "4.7k" V 8257 3251 40  0000 C CNN
 F 2 "" V 8180 3250 30  0000 C CNN
@@
 $EndComp
 $Comp
-L R R29
+L R R31
 U 1 1 53500D64
 P 8450 3250
-F 0 "R29" V 8530 3250 40  0000 C CNN
+F 0 "R31" V 8530 3250 40  0000 C CNN
 F 1 "4.7k" V 8457 3251 40  0000 C CNN
 F 2 "" V 8380 3250 30  0000 C CNN
@@
 $EndComp
 $Comp
-L R R30
+L R R32
 U 1 1 53500D6F
 P 8650 3250
-F 0 "R30" V 8730 3250 40  0000 C CNN
+F 0 "R32" V 8730 3250 40  0000 C CNN
 F 1 "4.7k" V 8657 3251 40  0000 C CNN
 F 2 "" V 8580 3250 30  0000 C CNN
@@
 All LEDs on this sheet 0603 Green\nType Osram lg_l29k\n
 $Comp
-L DIODE D10
+L DIODE D12
 U 1 1 535114A1
 P 3700 4650
-F 0 "D10" H 3700 4750 40  0000 C CNN
+F 0 "D12" H 3700 4750 40  0000 C CNN
 F 1 "DIODE" H 3700 4550 40  0000 C CNN
 F 2 "" H 3700 4650 60  0000 C CNN
@@
 	3700 4900 3700 4850
 $Comp
-L DIODE D11
+L DIODE D13
 U 1 1 535115D5
 P 3750 2400
-F 0 "D11" H 3750 2500 40  0000 C CNN
+F 0 "D13" H 3750 2500 40  0000 C CNN
 F 1 "DIODE" H 3750 2300 40  0000 C CNN
 F 2 "" H 3750 2400 60  0000 C CNN
@@
 	3850 2100 3850 2300
 $Comp
-L DIODE D15
+L DIODE D17
 U 1 1 53511841
 P 4750 3050
-F 0 "D15" H 4750 3150 40  0000 C CNN
+F 0 "D17" H 4750 3150 40  0000 C CNN
 F 1 "DIODE" H 4750 2950 40  0000 C CNN
 F 2 "" H 4750 3050 60  0000 C CNN
@@
 Connection ~ 3700 4900
 $Comp
-L DIODE D14
+L DIODE D16
 U 1 1 53511B29
 P 4650 5300
-F 0 "D14" H 4650 5400 40  0000 C CNN
+F 0 "D16" H 4650 5400 40  0000 C CNN
 F 1 "DIODE" H 4650 5200 40  0000 C CNN
 F 2 "" H 4650 5300 60  0000 C CNN
